Commit message: changed go2 parameters to match model, but still no odom

File: tbai_description/urdf/robot_single_realsense.xacro (robot description, xacro)
@@ -2,9 +2,8 @@
 <robot name="go2" xmlns:xacro="http://www.ros.org/wiki/xacro">
     <xacro:arg name="DEBUG" default="false"/>
-    <xacro:include filename="$(find go2_description)/xacro/const.xacro"/>
-    <xacro:include filename="$(find go2_description)/xacro/materials.xacro"/>
-    <xacro:include filename="$(find go2_description)/xacro/leg.xacro"/>
-    <!-- <xacro:include filename="$(find go2_description)/xacro/stairs.xacro"/> -->
-    <xacro:include filename="$(find go2_description)/xacro/gazebo.xacro"/>
+    <xacro:include filename="$(find tbai_description)/xacro/const.xacro"/>
+    <xacro:include filename="$(find tbai_description)/xacro/materials.xacro"/>
+    <xacro:include filename="$(find tbai_description)/xacro/leg.xacro"/>
+    <xacro:include filename="$(find tbai_description)/xacro/gazebo.xacro"/>
     <!-- <xacro:include filename="$(find go2_gazebo)/launch/stairs.urdf.xacro"/> -->
     <!-- <xacro:stairs stairs="15" xpos="0" ypos="0" zpos="0" /> -->
@@ -37,5 +36,5 @@
             <origin rpy="0 0 0" xyz="0 0 0"/>
             <geometry>
-                <mesh filename="package://go2_description/meshes/trunk.dae" scale="1 1 1"/>
+                <mesh filename="package://tbai_description/meshes/trunk.dae" scale="1 1 1"/>
             </geometry>
             <!-- <material name="orange"/> -->
@@ -113,5 +112,5 @@
     <xacro:leg name="RL" mirror="1"  mirror_dae="True"   front_hind="-1" front_hind_dae="False" />
     <!-- RealSense D435 -->
-    <xacro:include filename="$(find go2_description)/xacro/_d435.urdf.xacro" />
+    <xacro:include filename="$(find tbai_description)/xacro/_d435.urdf.xacro" />
     <xacro:sensor_d435 parent="base" name="camera" topics_ns="camera">
       <origin xyz="0.3 0 0.075" rpy="0 0.50 0" />
