Commit message: modeling new go2 urdf off of anymal

File: go2_description/xacro/robot_single_realsense.xacro (robot description, xacro)
@@ -5,10 +5,22 @@
     <xacro:include filename="$(find go2_description)/xacro/materials.xacro"/>
     <xacro:include filename="$(find go2_description)/xacro/leg.xacro"/>
-    <!-- <xacro:include filename="$(find go2_description)/xacro/stairs.xacro"/> -->
-    <xacro:include filename="$(find go2_description)/xacro/gazebo.xacro"/>
-    <!-- <xacro:include filename="$(find go2_gazebo)/launch/stairs.urdf.xacro"/> -->
-    <!-- <xacro:stairs stairs="15" xpos="0" ypos="0" zpos="0" /> -->
-    <!-- Rotor related joint and link is only for demonstrate location. -->
-    <!-- Actually, the rotor will rotate and the joint is not fixed. Reduction ratio should be considered. -->
+    <!-- <xacro:include filename="$(find go2_description)/xacro/gazebo.xacro"/> -->
+    <xacro:include filename="$(find tbai_description)/urdf/utils.xacro" />
+    <!-- Transmissions LF -->
+    <xacro:transmission name="transmission_LF_HAA" joint="LF_HAA" actuator="motor_LF_HAA"/>
+    <xacro:transmission name="transmission_LF_HFE" joint="LF_HFE" actuator="motor_LF_HFE"/>
+    <xacro:transmission name="transmission_LF_KFE" joint="LF_KFE" actuator="motor_LF_KFE"/>
+    <!-- Transmissions LH -->
+    <xacro:transmission name="transmission_LH_HAA" joint="LH_HAA" actuator="motor_LH_HAA"/>
+    <xacro:transmission name="transmission_LH_HFE" joint="LH_HFE" actuator="motor_LH_HFE"/>
+    <xacro:transmission name="transmission_LH_KFE" joint="LH_KFE" actuator="motor_LH_KFE"/>
+    <!-- Transmissions RF -->
+    <xacro:transmission name="transmission_RF_HAA" joint="RF_HAA" actuator="motor_RF_HAA"/>
+    <xacro:transmission name="transmission_RF_HFE" joint="RF_HFE" actuator="motor_RF_HFE"/>
+    <xacro:transmission name="transmission_RF_KFE" joint="RF_KFE" actuator="motor_RF_KFE"/>
+    <!-- Transmissions RH -->
+    <xacro:transmission name="transmission_RH_HAA" joint="RH_HAA" actuator="motor_RH_HAA"/>
+    <xacro:transmission name="transmission_RH_HFE" joint="RH_HFE" actuator="motor_RH_HFE"/>
+    <xacro:transmission name="transmission_RH_KFE" joint="RH_KFE" actuator="motor_RH_KFE"/>
     <!-- Joint controller -->
     <gazebo>
@@ -128,3 +140,62 @@
       <origin xyz="0.3 0 0.075" rpy="0 0.50 0" />
     </xacro:sensor_d435>
+    <!-- Grabbing from tbai_description -->
+    <!-- Add contact sensors -->
+    <gazebo reference="LF_FOOT">
+        <sensor name="lf_foot_contact" type="contact">
+        <plugin name="lf_contact_plugin" filename="libContactSensor.so"/>
+        <contact>
+            <collision>LF_SHANK_fixed_joint_lump__LF_FOOT_collision_3</collision>
+        </contact>
+        </sensor>
+    </gazebo>
+    <gazebo reference="RF_FOOT">
+        <sensor name="rf_foot_contact" type="contact">
+        <plugin name="rf_contact_plugin" filename="libContactSensor.so"/>
+        <contact>
+            <collision>RF_SHANK_fixed_joint_lump__RF_FOOT_collision_3</collision>
+        </contact>
+        </sensor>
+    </gazebo>
+    <gazebo reference="LH_FOOT">
+        <sensor name="lh_foot_contact" type="contact">
+        <plugin name="lh_contact_plugin" filename="libContactSensor.so"/>
+        <contact>
+            <collision>LH_SHANK_fixed_joint_lump__LH_FOOT_collision_3</collision>
+        </contact>
+        </sensor>
+    </gazebo>
+    <gazebo reference="RH_FOOT">
+        <sensor name="rh_foot_contact" type="contact">
+        <plugin name="rh_contact_plugin" filename="libContactSensor.so"/>
+        <contact>
+            <collision>RH_SHANK_fixed_joint_lump__RH_FOOT_collision_3</collision>
+        </contact>
+        </sensor>
+    </gazebo>
+    <!-- Gazebo materials -->
+    <gazebo reference="LF_FOOT">
+        <mu1>1.85</mu1>
+        <mu2>1.85</mu2>
+        <kp value="1000000.0"/>
+        <kd value="100.0"/>
+    </gazebo>
+    <gazebo reference="RF_FOOT">
+        <mu1>1.85</mu1>
+        <mu2>1.85</mu2>
+        <kp value="1000000.0"/>
+        <kd value="100.0"/>
+    </gazebo>
+    <gazebo reference="LH_FOOT">
+        <mu1>1.85</mu1>
+        <mu2>1.85</mu2>
+        <kp value="1000000.0"/>
+        <kd value="100.0"/>
+    </gazebo>
+    <gazebo reference="RH_FOOT">
+        <mu1>1.85</mu1>
+        <mu2>1.85</mu2>
+        <kp value="1000000.0"/>
+        <kd value="100.0"/>
+    </gazebo>
 </robot>

File: tbai_description/urdf/anymal_d_gazebo.urdf.xacro (robot description, xacro)
@@ -1,36 +1,36 @@
 <?xml version="1.0"?>
 <robot xmlns:xacro="http://www.ros.org/wiki/xacro" name="anymal_d">
-<!-- Includes -->
-<xacro:include filename="utils.xacro" />
-<!-- Anymal D bare urdf -->
-<xacro:include filename="$(find ocs2_robotic_assets)/resources/anymal_d/urdf/anymal.urdf" />
-<!-- Transmissions LF -->
-<xacro:transmission name="transmission_LF_HAA" joint="LF_HAA" actuator="motor_LF_HAA"/>
-<xacro:transmission name="transmission_LF_HFE" joint="LF_HFE" actuator="motor_LF_HFE"/>
-<xacro:transmission name="transmission_LF_KFE" joint="LF_KFE" actuator="motor_LF_KFE"/>
-<!-- Transmissions LH -->
-<xacro:transmission name="transmission_LH_HAA" joint="LH_HAA" actuator="motor_LH_HAA"/>
-<xacro:transmission name="transmission_LH_HFE" joint="LH_HFE" actuator="motor_LH_HFE"/>
-<xacro:transmission name="transmission_LH_KFE" joint="LH_KFE" actuator="motor_LH_KFE"/>
-<!-- Transmissions RF -->
-<xacro:transmission name="transmission_RF_HAA" joint="RF_HAA" actuator="motor_RF_HAA"/>
-<xacro:transmission name="transmission_RF_HFE" joint="RF_HFE" actuator="motor_RF_HFE"/>
-<xacro:transmission name="transmission_RF_KFE" joint="RF_KFE" actuator="motor_RF_KFE"/>
-<!-- Transmissions RH -->
-<xacro:transmission name="transmission_RH_HAA" joint="RH_HAA" actuator="motor_RH_HAA"/>
-<xacro:transmission name="transmission_RH_HFE" joint="RH_HFE" actuator="motor_RH_HFE"/>
-<xacro:transmission name="transmission_RH_KFE" joint="RH_KFE" actuator="motor_RH_KFE"/>
-<!-- Joint controller -->
-<gazebo>
-  <plugin filename="libgazebo_ros_control.so" name="gazebo_ros_control">
-    <robotSimType>gazebo_ros_control/DefaultRobotHWSim</robotSimType>
-    <robotNamespace>/anymal_d</robotNamespace>
-  </plugin>
-</gazebo>
-<!-- State publisher -->
-<gazebo>
-  <plugin filename="libStatePublisher.so" name="StatePublisher"/>
-</gazebo>
- <joint name="face_front_to_depth_camera_front_camera" type="fixed">
+    <!-- Includes -->
+    <xacro:include filename="utils.xacro" />
+    <!-- Anymal D bare urdf -->
+    <xacro:include filename="$(find ocs2_robotic_assets)/resources/anymal_d/urdf/anymal.urdf" />
+    <!-- Transmissions LF -->
+    <xacro:transmission name="transmission_LF_HAA" joint="LF_HAA" actuator="motor_LF_HAA"/>
+    <xacro:transmission name="transmission_LF_HFE" joint="LF_HFE" actuator="motor_LF_HFE"/>
+    <xacro:transmission name="transmission_LF_KFE" joint="LF_KFE" actuator="motor_LF_KFE"/>
+    <!-- Transmissions LH -->
+    <xacro:transmission name="transmission_LH_HAA" joint="LH_HAA" actuator="motor_LH_HAA"/>
+    <xacro:transmission name="transmission_LH_HFE" joint="LH_HFE" actuator="motor_LH_HFE"/>
+    <xacro:transmission name="transmission_LH_KFE" joint="LH_KFE" actuator="motor_LH_KFE"/>
+    <!-- Transmissions RF -->
+    <xacro:transmission name="transmission_RF_HAA" joint="RF_HAA" actuator="motor_RF_HAA"/>
+    <xacro:transmission name="transmission_RF_HFE" joint="RF_HFE" actuator="motor_RF_HFE"/>
+    <xacro:transmission name="transmission_RF_KFE" joint="RF_KFE" actuator="motor_RF_KFE"/>
+    <!-- Transmissions RH -->
+    <xacro:transmission name="transmission_RH_HAA" joint="RH_HAA" actuator="motor_RH_HAA"/>
+    <xacro:transmission name="transmission_RH_HFE" joint="RH_HFE" actuator="motor_RH_HFE"/>
+    <xacro:transmission name="transmission_RH_KFE" joint="RH_KFE" actuator="motor_RH_KFE"/>
+    <!-- Joint controller -->
+    <gazebo>
+    <plugin filename="libgazebo_ros_control.so" name="gazebo_ros_control">
+        <robotSimType>gazebo_ros_control/DefaultRobotHWSim</robotSimType>
+        <robotNamespace>/anymal_d</robotNamespace>
+    </plugin>
+    </gazebo>
+    <!-- State publisher -->
+    <gazebo>
+    <plugin filename="libStatePublisher.so" name="StatePublisher"/>
+    </gazebo>
+    <joint name="face_front_to_depth_camera_front_camera" type="fixed">
         <parent link="face_front"/>
         <child link="depth_camera_front_camera"/>
@@ -129,269 +129,269 @@
     <link name="depth_camera_rear_color_optical_frame"/>
     <!-- Camera joint -->
-  <!-- Front camera -->
-<!-- Front depth camera -->
-<gazebo reference="depth_camera_front_camera">
-<sensor type="depth" name="realsense_R200">
-    <always_on>true</always_on>
-    <visualize>false</visualize>
-    <update_rate>3</update_rate>
-    <camera>
-        <horizontal_fov>2.0</horizontal_fov>
-        <image>
-            <width>640</width>
-            <height>480</height>
-            <format>R8G8B8</format>
-        </image>
-        <depth_camera></depth_camera>
-        <clip>
-            <near>0.2</near>
-            <far>3</far>
-        </clip>
-        <noise>
-          <type>gaussian</type>
-          <mean>0.0</mean>
-          <stddev>0.05</stddev>
-        </noise>
-    </camera>
-    <plugin name="camera_controller" filename="libgazebo_ros_openni_kinect.so">
-    <baseline>0.2</baseline>
-    <alwaysOn>true</alwaysOn>
-    <updateRate>0.0</updateRate>
-    <cameraName>camera</cameraName>
-    <frameName>depth_camera_front_depth_optical_frame</frameName>
-    <imageTopicName>rgb/image_raw</imageTopicName>
-    <depthImageTopicName>depth/image_raw</depthImageTopicName>
-    <pointCloudTopicName>depth/points</pointCloudTopicName>
-    <cameraInfoTopicName>rgb/camera_info</cameraInfoTopicName>
-    <depthImageCameraInfoTopicName>depth/camera_info</depthImageCameraInfoTopicName>
-    <pointCloudCutoff>0.4</pointCloudCutoff>
-    <pointCloudCutoffMax>3.0</pointCloudCutoffMax>
-        <hackBaseline>0.07</hackBaseline>
-        <distortionK1>0.0</distortionK1>
-        <distortionK2>0.0</distortionK2>
-        <distortionK3>0.0</distortionK3>
-        <distortionT1>0.0</distortionT1>
-        <distortionT2>0.0</distortionT2>
-    <CxPrime>0.0</CxPrime>
-    <Cx>0.0</Cx>
-    <Cy>0.0</Cy>
-    <focalLength>0</focalLength>
-    <hackBaseline>0</hackBaseline>
-    </plugin>
-</sensor>
-</gazebo>
-<!-- Back camera -->
-<!-- Back depth camera -->
-<gazebo reference="depth_camera_rear_camera">
-<sensor type="depth" name="realsense_R200">
-    <always_on>true</always_on>
-    <visualize>false</visualize>
-    <update_rate>3</update_rate>
-    <camera>
-        <horizontal_fov>2.0</horizontal_fov>
-        <image>
-            <width>640</width>
-            <height>480</height>
-            <format>R8G8B8</format>
-        </image>
-        <depth_camera></depth_camera>
-        <clip>
-            <near>0.2</near>
-            <far>3</far>
-        </clip>
-        <noise>
-          <type>gaussian</type>
-          <mean>0.0</mean>
-          <stddev>0.05</stddev>
-        </noise>
-    </camera>
-    <plugin name="camera_controller" filename="libgazebo_ros_openni_kinect.so">
-    <baseline>0.2</baseline>
-    <alwaysOn>true</alwaysOn>
-    <updateRate>0.0</updateRate>
-    <cameraName>rear_camera</cameraName>
-    <frameName>depth_camera_rear_depth_optical_frame</frameName>
-    <imageTopicName>rgb/image_raw</imageTopicName>
-    <depthImageTopicName>depth/image_raw</depthImageTopicName>
-    <pointCloudTopicName>depth/points</pointCloudTopicName>
-    <cameraInfoTopicName>rgb/camera_info</cameraInfoTopicName>
-    <depthImageCameraInfoTopicName>depth/camera_info</depthImageCameraInfoTopicName>
-    <pointCloudCutoff>0.4</pointCloudCutoff>
-    <pointCloudCutoffMax>3.0</pointCloudCutoffMax>
-        <hackBaseline>0.07</hackBaseline>
-        <distortionK1>0.0</distortionK1>
-        <distortionK2>0.0</distortionK2>
-        <distortionK3>0.0</distortionK3>
-        <distortionT1>0.0</distortionT1>
-        <distortionT2>0.0</distortionT2>
-    <CxPrime>0.0</CxPrime>
-    <Cx>0.0</Cx>
-    <Cy>0.0</Cy>
-    <focalLength>0</focalLength>
-    <hackBaseline>0</hackBaseline>
-    </plugin>
-</sensor>
-</gazebo>
-<!-- Left camera -->
-<!-- Left depth camera -->
-<gazebo reference="depth_camera_left_camera">
-<sensor type="depth" name="realsense_R200">
-    <always_on>true</always_on>
-    <visualize>false</visualize>
-    <update_rate>3</update_rate>
-    <camera>
-        <horizontal_fov>2.0</horizontal_fov>
-        <image>
-            <width>640</width>
-            <height>480</height>
-            <format>R8G8B8</format>
-        </image>
-        <depth_camera></depth_camera>
-        <clip>
-            <near>0.2</near>
-            <far>3</far>
-        </clip>
-        <noise>
-          <type>gaussian</type>
-          <mean>0.0</mean>
-          <stddev>0.05</stddev>
-        </noise>
-    </camera>
-    <plugin name="camera_controller" filename="libgazebo_ros_openni_kinect.so">
-    <baseline>0.2</baseline>
-    <alwaysOn>true</alwaysOn>
-    <updateRate>0.0</updateRate>
-    <cameraName>left_camera</cameraName>
-    <frameName>depth_camera_left_depth_optical_frame</frameName>
-    <imageTopicName>rgb/image_raw</imageTopicName>
-    <depthImageTopicName>depth/image_raw</depthImageTopicName>
-    <pointCloudTopicName>depth/points</pointCloudTopicName>
-    <cameraInfoTopicName>rgb/camera_info</cameraInfoTopicName>
-    <depthImageCameraInfoTopicName>depth/camera_info</depthImageCameraInfoTopicName>
-    <pointCloudCutoff>0.4</pointCloudCutoff>
-    <pointCloudCutoffMax>3.0</pointCloudCutoffMax>
-        <hackBaseline>0.07</hackBaseline>
-        <distortionK1>0.0</distortionK1>
-        <distortionK2>0.0</distortionK2>
-        <distortionK3>0.0</distortionK3>
-        <distortionT1>0.0</distortionT1>
-        <distortionT2>0.0</distortionT2>
-    <CxPrime>0.0</CxPrime>
-    <Cx>0.0</Cx>
-    <Cy>0.0</Cy>
-    <focalLength>0</focalLength>
-    <hackBaseline>0</hackBaseline>
-    </plugin>
-</sensor>
-</gazebo>
-<!-- Right camera -->
-<!-- Right depth camera -->
-<gazebo reference="depth_camera_right_camera">
-<sensor type="depth" name="realsense_R200">
-    <always_on>true</always_on>
-    <visualize>false</visualize>
-    <update_rate>3</update_rate>
-    <camera>
-        <horizontal_fov>2.0</horizontal_fov>
-        <image>
-            <width>640</width>
-            <height>480</height>
-            <format>R8G8B8</format>
-        </image>
-        <depth_camera></depth_camera>
-        <clip>
-            <near>0.2</near>
-            <far>3</far>
-        </clip>
-        <noise>
-          <type>gaussian</type>
-          <mean>0.0</mean>
-          <stddev>0.05</stddev>
-        </noise>
-    </camera>
-    <plugin name="camera_controller" filename="libgazebo_ros_openni_kinect.so">
-    <baseline>0.2</baseline>
-    <alwaysOn>true</alwaysOn>
-    <updateRate>0.0</updateRate>
-    <cameraName>right_camera</cameraName>
-    <frameName>depth_camera_right_depth_optical_frame</frameName>
-    <imageTopicName>rgb/image_raw</imageTopicName>
-    <depthImageTopicName>depth/image_raw</depthImageTopicName>
-    <pointCloudTopicName>depth/points</pointCloudTopicName>
-    <cameraInfoTopicName>rgb/camera_info</cameraInfoTopicName>
-    <depthImageCameraInfoTopicName>depth/camera_info</depthImageCameraInfoTopicName>
-    <pointCloudCutoff>0.4</pointCloudCutoff>
-    <pointCloudCutoffMax>3.0</pointCloudCutoffMax>
-        <hackBaseline>0.07</hackBaseline>
-        <distortionK1>0.0</distortionK1>
-        <distortionK2>0.0</distortionK2>
-        <distortionK3>0.0</distortionK3>
-        <distortionT1>0.0</distortionT1>
-        <distortionT2>0.0</distortionT2>
-    <CxPrime>0.0</CxPrime>
-    <Cx>0.0</Cx>
-    <Cy>0.0</Cy>
-    <focalLength>0</focalLength>
-    <hackBaseline>0</hackBaseline>
-    </plugin>
-</sensor>
-</gazebo>
-<!-- Add contact sensors -->
-<gazebo reference="LF_FOOT">
-    <sensor name="lf_foot_contact" type="contact">
-    <plugin name="lf_contact_plugin" filename="libContactSensor.so"/>
-    <contact>
-        <collision>LF_SHANK_fixed_joint_lump__LF_FOOT_collision_3</collision>
-    </contact>
-    </sensor>
-</gazebo>
-<gazebo reference="RF_FOOT">
-    <sensor name="rf_foot_contact" type="contact">
-    <plugin name="rf_contact_plugin" filename="libContactSensor.so"/>
-    <contact>
-        <collision>RF_SHANK_fixed_joint_lump__RF_FOOT_collision_3</collision>
-    </contact>
-    </sensor>
-</gazebo>
-<gazebo reference="LH_FOOT">
-    <sensor name="lh_foot_contact" type="contact">
-    <plugin name="lh_contact_plugin" filename="libContactSensor.so"/>
-    <contact>
-        <collision>LH_SHANK_fixed_joint_lump__LH_FOOT_collision_3</collision>
-    </contact>
-    </sensor>
-</gazebo>
-<gazebo reference="RH_FOOT">
-    <sensor name="rh_foot_contact" type="contact">
-    <plugin name="rh_contact_plugin" filename="libContactSensor.so"/>
-    <contact>
-        <collision>RH_SHANK_fixed_joint_lump__RH_FOOT_collision_3</collision>
-    </contact>
-    </sensor>
-</gazebo>
-<!-- Gazebo materials -->
-<gazebo reference="LF_FOOT">
-  <mu1>1.85</mu1>
-  <mu2>1.85</mu2>
-  <kp value="1000000.0"/>
-  <kd value="100.0"/>
-</gazebo>
-<gazebo reference="RF_FOOT">
-  <mu1>1.85</mu1>
-  <mu2>1.85</mu2>
-  <kp value="1000000.0"/>
-  <kd value="100.0"/>
-</gazebo>
-<gazebo reference="LH_FOOT">
-  <mu1>1.85</mu1>
-  <mu2>1.85</mu2>
-  <kp value="1000000.0"/>
-  <kd value="100.0"/>
-</gazebo>
-<gazebo reference="RH_FOOT">
-  <mu1>1.85</mu1>
-  <mu2>1.85</mu2>
-  <kp value="1000000.0"/>
-  <kd value="100.0"/>
-</gazebo>
+    <!-- Front camera -->
+    <!-- Front depth camera -->
+    <gazebo reference="depth_camera_front_camera">
+        <sensor type="depth" name="realsense_R200">
+            <always_on>true</always_on>
+            <visualize>false</visualize>
+            <update_rate>3</update_rate>
+            <camera>
+                <horizontal_fov>2.0</horizontal_fov>
+                <image>
+                    <width>640</width>
+                    <height>480</height>
+                    <format>R8G8B8</format>
+                </image>
+                <depth_camera></depth_camera>
+                <clip>
+                    <near>0.2</near>
+                    <far>3</far>
+                </clip>
+                <noise>
+                <type>gaussian</type>
+                <mean>0.0</mean>
+                <stddev>0.05</stddev>
+                </noise>
+            </camera>
+            <plugin name="camera_controller" filename="libgazebo_ros_openni_kinect.so">
+            <baseline>0.2</baseline>
+            <alwaysOn>true</alwaysOn>
+            <updateRate>0.0</updateRate>
+            <cameraName>camera</cameraName>
+            <frameName>depth_camera_front_depth_optical_frame</frameName>
+            <imageTopicName>rgb/image_raw</imageTopicName>
+            <depthImageTopicName>depth/image_raw</depthImageTopicName>
+            <pointCloudTopicName>depth/points</pointCloudTopicName>
+            <cameraInfoTopicName>rgb/camera_info</cameraInfoTopicName>
+            <depthImageCameraInfoTopicName>depth/camera_info</depthImageCameraInfoTopicName>
+            <pointCloudCutoff>0.4</pointCloudCutoff>
+            <pointCloudCutoffMax>3.0</pointCloudCutoffMax>
+                <hackBaseline>0.07</hackBaseline>
+                <distortionK1>0.0</distortionK1>
+                <distortionK2>0.0</distortionK2>
+                <distortionK3>0.0</distortionK3>
+                <distortionT1>0.0</distortionT1>
+                <distortionT2>0.0</distortionT2>
+            <CxPrime>0.0</CxPrime>
+            <Cx>0.0</Cx>
+            <Cy>0.0</Cy>
+            <focalLength>0</focalLength>
+            <hackBaseline>0</hackBaseline>
+            </plugin>
+        </sensor>
+    </gazebo>
+    <!-- Back camera -->
+    <!-- Back depth camera -->
+    <gazebo reference="depth_camera_rear_camera">
+        <sensor type="depth" name="realsense_R200">
+            <always_on>true</always_on>
+            <visualize>false</visualize>
+            <update_rate>3</update_rate>
+            <camera>
+                <horizontal_fov>2.0</horizontal_fov>
+                <image>
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